Commit message: The wall as measured, the bar's collision fitted to its section, scans at 3.5 / 4.5 cm to try
At the scan's start the arm stood exactly at the build's joints, yet the
paper was 17.2 cm from the flange where the build put 10.74: the new wall
is 6.46 cm further than the placeholder canvas. The first scans were thus
~13 cm from the LED chips -- blurred (a bare LED's spot ~1.3 x the distance).

- Canvas and scan area moved back 6.46 cm along the canvas normal (both shows).
- uv_bar.urdf: the bar's middle, two strips above and below, the mount block
  and the plate as four strips, so each capsule hugs its part: 4.3 mm past
  the shade's rim (was 7.8), every one of the CAD's 17,459 points inside.
  strip_face's LED face is the tool's TCP (the shade's rim), not a box's top.
- Both shows rebuilt: every segment clear (bigwipe 87, party 85).
- build --scan-only --gap M: the scan alone at another gap, to
  shows/scans/<show>_gap<mm>/ (in git); 3.5 and 4.5 cm built (3.1 / 4.1 cm
  clear of the paper at the scan's 3 cm margin). show_stream --scan-test
  --scan-from DIR plays one (refused if built from other inputs);
  scan_test_ui's Distance picks it.

Co-Authored-By: Claude Opus 5.5 <noreply@anthropic.com>

File: assets/tools/uv_bar.urdf (robot description, URDF)
Before this commit: robot uv_bar, 4 links, 3 joints
Links:
- removed link bracket
- added link bracket_a; collision box size=0.029 0.119 0.018
- added link bracket_b; collision box size=0.029 0.119 0.018
- added link bracket_c; collision box size=0.029 0.119 0.018
- added link bracket_d; collision box size=0.029 0.119 0.018
- added link mount_a; collision box size=0.033 0.10 0.016
- added link mount_b; collision box size=0.033 0.10 0.016
- added link strip_bottom_a; collision box size=0.015 1.0875 0.0087
- added link strip_bottom_b; collision box size=0.015 1.0875 0.0087
- added link strip_top_a; collision box size=0.0145 1.0875 0.0094
- added link strip_top_b; collision box size=0.0145 1.0875 0.0094
- link strip: geometry collision box size=0.037 1.0875 0.018
Joints:
- removed joint tool_mount_to_bracket
- added joint tool_mount_to_bracket_a: type fixed, parent tool_mount, child bracket_a, origin xyz=0 0 0 rpy=0 0 0
- added joint tool_mount_to_bracket_b: type fixed, parent tool_mount, child bracket_b, origin xyz=0 0 0 rpy=0 0 0
- added joint tool_mount_to_bracket_c: type fixed, parent tool_mount, child bracket_c, origin xyz=0 0 0 rpy=0 0 0
- added joint tool_mount_to_bracket_d: type fixed, parent tool_mount, child bracket_d, origin xyz=0 0 0 rpy=0 0 0
- added joint tool_mount_to_mount_a: type fixed, parent tool_mount, child mount_a, origin xyz=0 0 0 rpy=0 0 0
- added joint tool_mount_to_mount_b: type fixed, parent tool_mount, child mount_b, origin xyz=0 0 0 rpy=0 0 0
- added joint tool_mount_to_strip_bottom_a: type fixed, parent tool_mount, child strip_bottom_a, origin xyz=0 0 0 rpy=0 0 0
- added joint tool_mount_to_strip_bottom_b: type fixed, parent tool_mount, child strip_bottom_b, origin xyz=0 0 0 rpy=0 0 0
- added joint tool_mount_to_strip_top_a: type fixed, parent tool_mount, child strip_top_a, origin xyz=0 0 0 rpy=0 0 0
- added joint tool_mount_to_strip_top_b: type fixed, parent tool_mount, child strip_top_b, origin xyz=0 0 0 rpy=0 0 0

Commit message: The party's scan at 2 mm: the bar's collision model hugs its front; the wall as taped
The 6.3 mm scan painted fine and measured 8 mm by tape at its start; the
user wants 2 mm, the tape the reference.

- The wall 1.7 mm further out in both configs, as the tape says (the bar
  pressed flat on it had sat a little in it).
- assets/tools/uv_bar.urdf: the bar's middle split into five boxes across,
  the shade into six, the lower strips 1.2 mm wider: the capsules reach
  0.93 mm past the shade's rim (was 4.3) and still hold all 17,459 CAD
  points -- cad_tool_mesh's self-test checks both. collision.strip_width:
  the scan's travel still uses the bar's 37 mm, not its middle strip's.
- scan.led_gap_m 0.002, margins.scan_canvas_m 0.0008 (the collision model
  1.1 mm off the paper); both shows rebuilt (85 / 87 segments).
- show.py build --area-height H (scan-only): a shorter picture, its top
  kept -- 0.5 m/s needs 0.8 m (the forearm by the floor at 1 m).
- Scan variants: 2 mm at 0.3 / 0.4 / 0.5 m/s (0.8 m tall), 4 / 8 / 35 mm;
  the older ones dropped (the tool changed).
- scan_test_ui: a half-typed number no longer stops the window (TclError
  on '.'); a step with no number refused, not guessed.
- collision's self-test: the bar is 1.0875 m with its caps (it asked for
  1.0 since the CAD bar came in).

Co-Authored-By: Claude Opus 5.5 <noreply@anthropic.com>

File: assets/tools/uv_bar.urdf (robot description, URDF)
Before this commit: robot uv_bar, 13 links, 12 joints
Links:
- removed link strip_top_a
- removed link strip_top_b
- added link strip_l1; collision box size=0.0074 1.0875 0.018
- added link strip_l2; collision box size=0.0074 1.0875 0.018
- added link strip_r1; collision box size=0.0074 1.0875 0.018
- added link strip_r2; collision box size=0.0074 1.0875 0.018
- added link strip_top_a1; collision box size=0.00483333 1.0875 0.0094
- added link strip_top_a2; collision box size=0.00483333 1.0875 0.0094
- added link strip_top_a3; collision box size=0.00483333 1.0875 0.0094
- added link strip_top_b1; collision box size=0.00483333 1.0875 0.0094
- added link strip_top_b2; collision box size=0.00483333 1.0875 0.0094
- added link strip_top_b3; collision box size=0.00483333 1.0875 0.0094
- link strip: geometry collision box size=0.0074 1.0875 0.018
- link strip_bottom_a: geometry collision box size=0.0162 1.0875 0.0087
- link strip_bottom_b: geometry collision box size=0.0162 1.0875 0.0087
Joints:
- removed joint tool_mount_to_strip_top_a
- removed joint tool_mount_to_strip_top_b
- added joint tool_mount_to_strip_l1: type fixed, parent tool_mount, child strip_l1, origin xyz=0 0 0 rpy=0 0 0
- added joint tool_mount_to_strip_l2: type fixed, parent tool_mount, child strip_l2, origin xyz=0 0 0 rpy=0 0 0
- added joint tool_mount_to_strip_r1: type fixed, parent tool_mount, child strip_r1, origin xyz=0 0 0 rpy=0 0 0
- added joint tool_mount_to_strip_r2: type fixed, parent tool_mount, child strip_r2, origin xyz=0 0 0 rpy=0 0 0
- added joint tool_mount_to_strip_top_a1: type fixed, parent tool_mount, child strip_top_a1, origin xyz=0 0 0 rpy=0 0 0
- added joint tool_mount_to_strip_top_a2: type fixed, parent tool_mount, child strip_top_a2, origin xyz=0 0 0 rpy=0 0 0
- added joint tool_mount_to_strip_top_a3: type fixed, parent tool_mount, child strip_top_a3, origin xyz=0 0 0 rpy=0 0 0
- added joint tool_mount_to_strip_top_b1: type fixed, parent tool_mount, child strip_top_b1, origin xyz=0 0 0 rpy=0 0 0
- added joint tool_mount_to_strip_top_b2: type fixed, parent tool_mount, child strip_top_b2, origin xyz=0 0 0 rpy=0 0 0
- added joint tool_mount_to_strip_top_b3: type fixed, parent tool_mount, child strip_top_b3, origin xyz=0 0 0 rpy=0 0 0
